File: hardware/joysticks_right.sch (EAGLE design)
At the start: 8 parts, among them IC1 MEGA16-M

Commit message: added mode selection jumper (SPI/I2C)
Parts:
- added SV2: (no value), con-lstb:MA03-1
Connections:
- new net MD_SEL: IC1.(OC1A)PD5, SV2.2
- net GND: now also SV2.3
- net VCC: now also SV2.1
Other:
- moved on the sheet: JOY_RB, JOY_RT, SV1

Commit message: set value for xtal-caps
Parts:
- C1, C2: value (none) -> 18p
Changed lines of the file:
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@@
 <part name="P+1" library="supply1" deviceset="VCC" device=""/>
 <part name="U$1" library="jocki" deviceset="CRYSTAL" device="ABM2"/>
-<part name="C1" library="rcl" deviceset="C-EU" device="C0603"/>
-<part name="C2" library="rcl" deviceset="C-EU" device="C0603"/>
+<part name="C1" library="rcl" deviceset="C-EU" device="C0603" value="18p"/>
+<part name="C2" library="rcl" deviceset="C-EU" device="C0603" value="18p"/>
 <part name="GND2" library="supply1" deviceset="GND" device=""/>
 <part name="SV1" library="con-lstb" deviceset="MA05-2" device=""/>
